File: Hardware/KiCad/6_channel_esp32_energy_meter.sch (KiCad schematic (older format))
At the start: 0 parts

Commit message: Make the schematic not terrible.
Parts:
- added CF7: BLU, 6_channel_esp32_energy_meter:CHIPLED_0603, symbol 6_channel_esp32_energy_meter-eagle-import:LEDCHIPLED_0603
- added J1: Conn_02x05_Odd_Even, Connector_IDC:IDC-Header_2x05_P2.54mm_Vertical, symbol Connector_Generic:Conn_02x05_Odd_Even
- added J2: Conn_02x07_Odd_Even, Connector_IDC:IDC-Header_2x07_P2.54mm_Vertical, symbol Connector_Generic:Conn_02x07_Odd_Even
- added R47: 1k, 6_channel_esp32_energy_meter:R0603, symbol 6_channel_esp32_energy_meter-eagle-import:R-US_R0603
Connections:
- net labels added: +3.3V, GND
- wire segments 0 -> 73

Commit message: Working on layout.
Parts:
- added C1: 0.1uF, Capacitor_SMD:C_0603_1608Metric_Pad1.05x0.95mm_HandSolder, symbol Device:C
- added C2, C3: CP1, Capacitor_THT:CP_Radial_D12.5mm_P5.00mm, symbol Device:CP1
- added H1, H2, H3, H4, H5: MountingHole, MountingHole:MountingHole_3.2mm_M3_Pad_Via, symbol Mechanical:MountingHole
- added R1: 10K, Resistor_SMD:R_0603_1608Metric_Pad1.05x0.95mm_HandSolder, symbol Device:R
- R2: renamed from R47; footprint 6_channel_esp32_energy_meter:R0603 -> Resistor_SMD:R_0603_1608Metric_Pad1.05x0.95mm_HandSolder
- renumbered CF7 to CF1
Connections:
- wire segments 73 -> 95
- no-connect marks 0 -> 2

Commit message: Minor footprint cleanup.
Connections:
- wire segments 95 -> 96
Changed lines of the file:
@@
 	3200 1700 2900 1700
 Wire Wire Line
-	2900 1700 2900 2750
-Wire Wire Line
 	2900 3900 3200 3900
 Wire Wire Line
 	3200 4000 2950 4000
 Wire Wire Line
-	2950 4000 2950 2850
-Wire Wire Line
 	2950 1800 3200 1800
 Wire Wire Line
 	3200 2000 3050 2000
 Wire Wire Line
-	3050 2000 3050 3250
-Wire Wire Line
 	3050 4200 3200 4200
 Wire Wire Line
 	3200 4300 3100 4300
-Wire Wire Line
-	3100 4300 3100 3150
 Wire Wire Line
 	3100 2100 3200 2100
@@
 F 3 "~" H 1600 2750 50  0001 C CNN
 	1    1600 2750
-	1    0    0    -1
-$EndComp
-Wire Wire Line
-	1400 2650 1300 2650
-Wire Wire Line
-	1300 2650 1300 2550
-Wire Wire Line
-	1300 2550 1400 2550
-Wire Wire Line
-	1900 2550 2000 2550
-Wire Wire Line
-	2000 2550 2000 2650
-Wire Wire Line
-	2000 2650 1900 2650
-Wire Wire Line
-	1400 2850 1300 2850
-Wire Wire Line
-	1300 2850 1300 2950
-Wire Wire Line
-	1300 2950 1400 2950
-Wire Wire Line
-	1900 2850 2000 2850
-Wire Wire Line
-	2000 2850 2000 2950
-Wire Wire Line
-	2000 2950 1900 2950
-Wire Wire Line
-	2000 3150 2000 2950
-Connection ~ 2000 2950
-Wire Wire Line
-	1300 3250 1300 2950
-Connection ~ 1300 2950
-Wire Wire Line
-	2950 2850 2400 2850
-Wire Wire Line
-	1300 2550 1300 2250
-Wire Wire Line
-	1300 2250 2500 2250
-Wire Wire Line
-	2500 2250 2500 2750
-Wire Wire Line
-	2500 2750 2900 2750
-Connection ~ 1300 2550
-Wire Wire Line
-	2000 2550 2400 2550
-Wire Wire Line
-	2400 2550 2400 2850
-Connection ~ 2000 2550
+	1    0    0    1
+$EndComp
 $Comp
 L power:+3.3V #PWR03
@@
 	5550 4500 4800 4500
 Wire Wire Line
-	3050 3250 1300 3250
-Wire Wire Line
-	3100 3150 2000 3150
-Wire Wire Line
 	6600 3100 6650 3100
 Wire Wire Line
@@
 	1    0    0    -1
 $EndComp
-Connection ~ 2900 2750
-Wire Wire Line
-	2900 2750 2900 3900
-Connection ~ 2950 2850
-Wire Wire Line
-	2950 2850 2950 1800
-Connection ~ 3050 3250
-Wire Wire Line
-	3050 3250 3050 4200
-Connection ~ 3100 3150
-Wire Wire Line
-	3100 3150 3100 2100
 Wire Wire Line
 	6900 2900 6900 4100
@@
 	5500 1250 5500 1200
 Connection ~ 5500 1250
+Wire Wire Line
+	1400 2550 1350 2550
+Wire Wire Line
+	1350 2350 1950 2350
+Wire Wire Line
+	1950 2350 1950 2550
+Wire Wire Line
+	1950 2550 1900 2550
+Wire Wire Line
+	1350 2350 1350 2550
+Wire Wire Line
+	1400 2650 1250 2650
+Wire Wire Line
+	1250 2650 1250 2250
+Wire Wire Line
+	1250 2250 2050 2250
+Wire Wire Line
+	1900 2650 2050 2650
+Wire Wire Line
+	2050 2650 2050 2250
+Wire Wire Line
+	1400 2950 1350 2950
+Wire Wire Line
+	1350 2950 1350 3150
+Wire Wire Line
+	1350 3150 1950 3150
+Wire Wire Line
+	1950 3150 1950 2950
+Wire Wire Line
+	1950 2950 1900 2950
+Wire Wire Line
+	1900 2850 2050 2850
+Wire Wire Line
+	2050 2850 2050 3250
+Wire Wire Line
+	2050 3250 1250 3250
+Wire Wire Line
+	1250 3250 1250 2850
+Wire Wire Line
+	1250 2850 1400 2850
+Wire Wire Line
+	2900 1700 2900 2950
+Wire Wire Line
+	2950 1800 2950 2850
+Wire Wire Line
+	3050 2000 3050 2650
+Wire Wire Line
+	3100 2100 3100 2550
+Wire Wire Line
+	1950 2950 2900 2950
+Connection ~ 1950 2950
+Connection ~ 2900 2950
+Wire Wire Line
+	2900 2950 2900 3900
+Wire Wire Line
+	2950 2850 2050 2850
+Connection ~ 2950 2850
+Wire Wire Line
+	2950 2850 2950 4000
+Connection ~ 2050 2850
+Wire Wire Line
+	2050 2650 3050 2650
+Connection ~ 2050 2650
+Connection ~ 3050 2650
+Wire Wire Line
+	3050 2650 3050 4200
+Wire Wire Line
+	1950 2550 3100 2550
+Connection ~ 1950 2550
+Connection ~ 3100 2550
+Wire Wire Line
+	3100 2550 3100 4300
 $EndSCHEMATC
