File: Hardware/KiCad/single_metering_ic.sch (KiCad schematic (older format))
At the start: 58 parts, among them IC1 ATM90E36, Y1 16.384MHz

Commit message: Working on layout.
Parts:
- removed C1: 18nF, 6_channel_esp32_energy_meter:C0603, symbol Device:C
- removed C2, C3: .33uF, 6_channel_esp32_energy_meter:C0603, symbol Device:C
- removed R1, R2: 20K, Resistor_SMD:R_0603_1608Metric_Pad1.05x0.95mm_HandSolder, symbol Device:R
- added C18, C19: 10uF, Capacitor_SMD:C_1206_3216Metric_Pad1.42x1.75mm_HandSolder, symbol Device:C
- added C20, C21: 0.1uF, Capacitor_SMD:C_0603_1608Metric_Pad1.05x0.95mm_HandSolder, symbol Device:C
- added R24: 1K, Resistor_SMD:R_0603_1608Metric_Pad1.05x0.95mm_HandSolder, symbol Device:R
- C10, C5, C9: value 18nF -> 0.33uF; footprint 6_channel_esp32_energy_meter:C0603 -> Capacitor_SMD:C_0603_1608Metric_Pad1.05x0.95mm_HandSolder
- C11: value 0.1uF -> 0.33uF; footprint 6_channel_esp32_energy_meter:C0603 -> Capacitor_SMD:C_0603_1608Metric_Pad1.05x0.95mm_HandSolder
- C12: value 10uF -> 18nF; footprint 6_channel_esp32_energy_meter:C0603 -> Capacitor_SMD:C_0603_1608Metric_Pad1.05x0.95mm_HandSolder
- C13: value 0.1uF -> 18nF; footprint 6_channel_esp32_energy_meter:C0603 -> Capacitor_SMD:C_0603_1608Metric_Pad1.05x0.95mm_HandSolder
- C14: value 10uF -> 0.1uF; footprint 6_channel_esp32_energy_meter:C0603 -> Capacitor_SMD:C_0603_1608Metric_Pad1.05x0.95mm_HandSolder
- C15: value 0.1uF -> 10uF; footprint 6_channel_esp32_energy_meter:C0603 -> Capacitor_SMD:C_1206_3216Metric_Pad1.42x1.75mm_HandSolder
- C16, C17: footprint 6_channel_esp32_energy_meter:C0603 -> Capacitor_SMD:C_0603_1608Metric_Pad1.05x0.95mm_HandSolder
- C4, C8: value .33uF -> 18nF; footprint 6_channel_esp32_energy_meter:C0603 -> Capacitor_SMD:C_0603_1608Metric_Pad1.05x0.95mm_HandSolder
- C6, C7: value .33uF -> 0.33uF; footprint 6_channel_esp32_energy_meter:C0603 -> Capacitor_SMD:C_0603_1608Metric_Pad1.05x0.95mm_HandSolder
- R10, R11: value 100 -> 22R
- R12, R13, R14, R15: value 100 -> 100R
- R16, R17: value 1K -> 100R
- R18: value 10K -> 1K
- R19: value 220 -> 1K
- R20: value 10K -> 100R
- R21: value 1k -> 10K
- R22, R23: value 1k -> 1K
- R5: value 1K -> 20K
- R6: value 22 -> 20K
- R7, R8: value 22 -> 1K
- R9: value 1K -> 22R
- renumbered CF1 to CF2, CF2 to CF3, CF3 to CF4
Connections:
- net labels added: 1.8VDD, I1N, I1P, I2N, I2P, I3N, I3P
- wire segments 214 -> 213
- no-connect marks 0 -> 9
