File: Hardware/KiCad/Energy Monitor - Sensor PCB/Energy Monitor - Sensor PCB.sch (KiCad schematic (older format))
At the start: 13 parts, among them J1 Conn_02x05_Odd_Even, J2 Conn_02x07_Odd_Even

Commit message: This seems to be getting progressively more complicated. Library cleanup, moved everything to my system library.
Parts:
- CF1: symbol Energy-Monitor---Sensor-PCB-rescue:LEDCHIPLED_0603-6_channel_esp32_energy_meter-eagle-import-6_channel_esp32_energy_met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 -> custom:LEDCHIPLED_0603-6_channel_esp32_energy_meter-eagle-import-6_channel_esp32_energy_meter-rescue
- R2: symbol Energy-Monitor---Sensor-PCB-rescue:R-US_R0603-6_channel_esp32_energy_meter-eagle-import-6_channel_esp32_energy_meter-re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 -> custom:R-US_R0603-6_channel_esp32_energy_meter-eagle-import-6_channel_esp32_energy_meter-rescue
Connections:
- net +3V3: no longer J2.2 (Pin_2)
- new net +5V: J2.2 (Pin_2)
Other:
- note added: "5V Rail is unused on this board"
Changed lines of the file:
@@
 Wire Wire Line
 	6050 2700 6100 2700
-$Comp
-L power:+3.3V #PWR05
-U 1 1 5F43F22F
-P 6700 2650
-F 0 "#PWR05" H 6700 2500 50  0001 C CNN
-F 1 "+3.3V" H 6715 2823 50  0000 C CNN
-F 2 "" H 6700 2650 50  0001 C CNN
-F 3 "" H 6700 2650 50  0001 C CNN
-	1    6700 2650
-	1    0    0    -1
-$EndComp
 Wire Wire Line
 	6700 2650 6700 2700
@@
 	8300 4150 8300 4250
 $Comp
-L Energy-Monitor---Sensor-PCB-rescue:R-US_R0603-6_channel_esp32_energy_meter-eagle-import-6_channel_esp32_energy_meter-rescue R2
+L custom:R-US_R0603-6_channel_esp32_energy_meter-eagle-import-6_channel_esp32_energy_meter-rescue R2
 U 1 1 5F45F957
 P 8300 3950
@@
 $EndComp
 $Comp
-L Energy-Monitor---Sensor-PCB-rescue:LEDCHIPLED_0603-6_channel_esp32_energy_meter-eagle-import-6_channel_esp32_energy_meter-rescue CF1
+L custom:LEDCHIPLED_0603-6_channel_esp32_energy_meter-eagle-import-6_channel_esp32_energy_meter-rescue CF1
 U 1 1 5F45F95E
 P 8300 4350
@@
 NoConn ~ 1400 2750
 NoConn ~ 1900 2750
+$Comp
+L power:+5V #PWR?
+U 1 1 5F4680F3
+P 6700 2650
+F 0 "#PWR?" H 6700 2500 50  0001 C CNN
+F 1 "+5V" H 6715 2823 50  0000 C CNN
+F 2 "" H 6700 2650 50  0001 C CNN
+F 3 "" H 6700 2650 50  0001 C CNN
+	1    6700 2650
+	1    0    0    -1
+$EndComp
+Text Notes 5600 2100 0    50   ~ 0
+5V Rail is unused on this board
 $EndSCHEMATC
