File: Hardware/KiCad/Energy Monitor - Sensor PCB/single_metering_ic.sch (KiCad schematic (older format))
At the start: 58 parts, among them IC1 ATM90E36, Y1 16.384MHz

Commit message: Project cleanup. Kicad has too many garbage files it sprays everywhere.
Parts:
- CF2, CF3, CF4: symbol 6_channel_esp32_energy_meter-eagle-import:LEDCHIPLED_0603 -> Energy-Monitor---Sensor-PCB-rescue:LEDCHIPLED_0603-6_channel_esp32_energy_meter-eagle-import-6_channel_esp32_energy_met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
- CT1, CT2, CT3: symbol 6_channel_esp32_energy_meter-eagle-import:CONN_023.5MM -> Energy-Monitor---Sensor-PCB-rescue:CONN_023.5MM-6_channel_esp32_energy_meter-eagle-import-6_channel_esp32_energy_meter-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
- CT1-1, CT2-1, CT3-1: symbol 6_channel_esp32_energy_meter-eagle-import:SJ2-35813B-SMT-TR -> Energy-Monitor---Sensor-PCB-rescue:SJ2-35813B-SMT-TR-6_channel_esp32_energy_meter-eagle-import-6_channel_esp32_energy_m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
- IC1: symbol 6_channel_esp32_energy_meter-eagle-import:ATM90E36 -> Energy-Monitor---Sensor-PCB-rescue:ATM90E36-6_channel_esp32_energy_meter-eagle-import
- Y1: symbol 6_channel_esp32_energy_meter-eagle-import:CRYSTAL-GROUNDEDSMD-3.2X2.5 -> Energy-Monitor---Sensor-PCB-rescue:CRYSTAL-GROUNDEDSMD-3.2X2.5-6_channel_esp32_energy_meter-eagle-import
- ZX1, ZX2, ZX3, ZX4, ZX5, ZX6, ZX7: symbol 6_channel_esp32_energy_meter-eagle-import:WIREPADSMD1,27-254 -> Energy-Monitor---Sensor-PCB-rescue:WIREPADSMD1,27-254-6_channel_esp32_energy_meter-eagle-import-6_channel_esp32_energy_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

Commit message: This seems to be getting progressively more complicated. Library cleanup, moved everything to my system library.
Parts:
- CF2, CF3, CF4: symbol Energy-Monitor---Sensor-PCB-rescue:LEDCHIPLED_0603-6_channel_esp32_energy_meter-eagle-import-6_channel_esp32_energy_met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 -> custom:LEDCHIPLED_0603-6_channel_esp32_energy_meter-eagle-import-6_channel_esp32_energy_meter-rescue
- CT1, CT2, CT3: symbol Energy-Monitor---Sensor-PCB-rescue:CONN_023.5MM-6_channel_esp32_energy_meter-eagle-import-6_channel_esp32_energy_meter-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 -> custom:CONN_023.5MM-6_channel_esp32_energy_meter-eagle-import-6_channel_esp32_energy_meter-rescue
- CT1-1, CT2-1, CT3-1: symbol Energy-Monitor---Sensor-PCB-rescue:SJ2-35813B-SMT-TR-6_channel_esp32_energy_meter-eagle-import-6_channel_esp32_energy_m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 -> custom:SJ2-35813B-SMT-TR-6_channel_esp32_energy_meter-eagle-import-6_channel_esp32_energy_meter-rescue
- IC1: symbol Energy-Monitor---Sensor-PCB-rescue:ATM90E36-6_channel_esp32_energy_meter-eagle-import -> custom:ATM90E36-6_channel_esp32_energy_meter-eagle-import
- Y1: symbol Energy-Monitor---Sensor-PCB-rescue:CRYSTAL-GROUNDEDSMD-3.2X2.5-6_channel_esp32_energy_meter-eagle-import -> custom:CRYSTAL-GROUNDEDSMD-3.2X2.5-6_channel_esp32_energy_meter-eagle-import
- ZX1, ZX2, ZX3, ZX4, ZX5, ZX6, ZX7: symbol Energy-Monitor---Sensor-PCB-rescue:WIREPADSMD1,27-254-6_channel_esp32_energy_meter-eagle-import-6_channel_esp32_energy_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 -> custom:WIREPADSMD1,27-254-6_channel_esp32_energy_meter-eagle-import-6_channel_esp32_energy_meter-rescue

Commit message: Switch to a better jack.
Parts:
- removed CT1-1, CT3-1: SJ2-35813B-SMT-TR, 6_channel_esp32_energy_meter:CUI_SJ2-35813B-SMT-TR, symbol custom:SJ2-35813B-SMT-TR-6_channel_esp32_energy_meter-eagle-import-6_channel_es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
- added CT1-1, CT3-1: SJ2-35813B-SMT-TR, custom:PJ-3270, symbol custom:PJ-3270
- CT2-1: footprint 6_channel_esp32_energy_meter:CUI_SJ2-35813B-SMT-TR -> custom:PJ-3270; symbol custom:SJ2-35813B-SMT-TR-6_channel_esp32_energy_meter-eagle-import-6_channel_esp32_energy_meter-rescue -> custom:PJ-3270
Connections:
- net at CT1.1, R12.1, R9.2: now also CT1-1.3 (SLEEVE)
- net at CT1.2, R13.1, R9.1: now also CT1-1.2 (TIP)
- net at CT2.1, R10.2, R14.1: now also CT2-1.3 (SLEEVE); no longer CT2-1.1 (SLEEVE)
- net at CT3.2, R11.1, R17.1: now also CT3-1.2 (TIP)
- net at CT3.1, R11.2, R16.1: now also CT3-1.3 (SLEEVE)
- no-connect marks 9 -> 12
Changed lines of the file:
@@
 $EndComp
 $Comp
-L custom:SJ2-35813B-SMT-TR-6_channel_esp32_energy_meter-eagle-import-6_channel_esp32_energy_meter-rescue CT1-?
-U 1 1 17D17B43
-P 1450 2300
-AR Path="/17D17B43" Ref="CT1-?"  Part="1"
-AR Path="/5F4280A7/17D17B43" Ref="CT1-1"  Part="1"
-AR Path="/5F53F374/17D17B43" Ref="CT1-2"  Part="1"
-AR Path="/5F541DC1/17D17B43" Ref="CT1-?"  Part="1"
-F 0 "CT1-1" H 1049 2701 85  0000 L BNN
-F 1 "SJ2-35813B-SMT-TR" H 1049 1899 85  0000 L BNN
-F 2 "6_channel_esp32_energy_meter:CUI_SJ2-35813B-SMT-TR" H 1450 2300 50  0001 C CNN
-F 3 "" H 1450 2300 50  0001 C CNN
-	1    1450 2300
-	1    0    0    -1
-$EndComp
-$Comp
-L custom:SJ2-35813B-SMT-TR-6_channel_esp32_energy_meter-eagle-import-6_channel_esp32_energy_meter-rescue CT2-?
+L custom:PJ-3270 CT2-?
 U 1 1 E89ABBD2
 P 1450 3500
@@
 F 0 "CT2-1" H 1049 3901 85  0000 L BNN
 F 1 "SJ2-35813B-SMT-TR" H 1049 3099 85  0000 L BNN
-F 2 "6_channel_esp32_energy_meter:CUI_SJ2-35813B-SMT-TR" H 1450 3500 50  0001 C CNN
+F 2 "custom:PJ-3270" H 1450 3500 50  0001 C CNN
 F 3 "" H 1450 3500 50  0001 C CNN
 	1    1450 3500
-	1    0    0    -1
-$EndComp
-$Comp
-L custom:SJ2-35813B-SMT-TR-6_channel_esp32_energy_meter-eagle-import-6_channel_esp32_energy_meter-rescue CT3-?
-U 1 1 F08860F8
-P 1450 4700
-AR Path="/F08860F8" Ref="CT3-?"  Part="1"
-AR Path="/5F4280A7/F08860F8" Ref="CT3-1"  Part="1"
-AR Path="/5F53F374/F08860F8" Ref="CT3-2"  Part="1"
-AR Path="/5F541DC1/F08860F8" Ref="CT3-?"  Part="1"
-F 0 "CT3-1" H 1049 5101 85  0000 L BNN
-F 1 "SJ2-35813B-SMT-TR" H 1049 4299 85  0000 L BNN
-F 2 "6_channel_esp32_energy_meter:CUI_SJ2-35813B-SMT-TR" H 1450 4700 50  0001 C CNN
-F 3 "" H 1450 4700 50  0001 C CNN
-	1    1450 4700
 	1    0    0    -1
 $EndComp
@@
 Wire Wire Line
 	7800 4200 9450 4200
+$Comp
+L custom:PJ-3270 CT2-?
+U 1 1 5F55E2FA
+P 1450 2300
+AR Path="/5F55E2FA" Ref="CT2-?"  Part="1"
+AR Path="/5F4280A7/5F55E2FA" Ref="CT1-1"  Part="1"
+AR Path="/5F53F374/5F55E2FA" Ref="CT1-2"  Part="1"
+AR Path="/5F541DC1/5F55E2FA" Ref="CT2-?"  Part="1"
+F 0 "CT1-1" H 1049 2701 85  0000 L BNN
+F 1 "SJ2-35813B-SMT-TR" H 1049 1899 85  0000 L BNN
+F 2 "custom:PJ-3270" H 1450 2300 50  0001 C CNN
+F 3 "" H 1450 2300 50  0001 C CNN
+	1    1450 2300
+	1    0    0    -1
+$EndComp
+$Comp
+L custom:PJ-3270 CT1-?
+U 1 1 5F56325B
+P 1450 4700
+AR Path="/5F56325B" Ref="CT1-?"  Part="1"
+AR Path="/5F4280A7/5F56325B" Ref="CT3-1"  Part="1"
+AR Path="/5F53F374/5F56325B" Ref="CT3-2"  Part="1"
+AR Path="/5F541DC1/5F56325B" Ref="CT1-?"  Part="1"
+F 0 "CT3-1" H 1049 5101 85  0000 L BNN
+F 1 "SJ2-35813B-SMT-TR" H 1049 4299 85  0000 L BNN
+F 2 "custom:PJ-3270" H 1450 4700 50  0001 C CNN
+F 3 "" H 1450 4700 50  0001 C CNN
+	1    1450 4700
+	1    0    0    -1
+$EndComp
+NoConn ~ 2050 2500
+NoConn ~ 2050 3700
+NoConn ~ 2050 4900
 $EndSCHEMATC
