File: Hardware/KiCad/Energy Monitor - ESP32 PCB/EnergyMonitor - ESP PCB.sch (KiCad schematic (older format))
At the start: 16 parts, among them J1 Conn_02x05_Odd_Even, J2 Conn_02x07_Odd_Even, J3 Conn_02x07_Odd_Even, J4 Conn_02x07_Odd_Even, J5 Conn_02x07_Odd_Even, J6 Conn_02x07_Odd_Even, J7 Conn_02x07_Odd_Even, U1 4072, U2 4072, U3 4072, U4 4072

Commit message: This seems to be getting progressively more complicated. Library cleanup, moved everything to my system library.
Parts:
- added C10, C11: 0.1 uF, Capacitor_SMD:C_0603_1608Metric_Pad1.05x0.95mm_HandSolder, symbol Device:C_Small
- added C12, C13, C8, C9: 22 uF, Capacitor_SMD:C_1206_3216Metric_Pad1.42x1.75mm_HandSolder, symbol Device:C_Small
- added C14, C4, C5: CP1, Capacitor_THT:CP_Radial_D12.5mm_P5.00mm, symbol Device:CP1
- added C15, C16: CP1, Capacitor_THT:CP_Radial_D8.0mm_P3.50mm, symbol Device:CP1
- added C6, C7: 10 uF, 35V, Capacitor_SMD:C_1206_3216Metric_Pad1.42x1.75mm_HandSolder, symbol Device:C_Small
- added H1, H2, H3, H4: MountingHole, MountingHole:MountingHole_3.2mm_M3_Pad_Via, symbol Mechanical:MountingHole
- added L1, L2, L3: 47 uH, Inductor_SMD:L_Bourns-SRU8028_8.0x8.0mm, symbol Device:L_Small
- added R3: 330R, Resistor_SMD:R_0603_1608Metric_Pad1.05x0.95mm_HandSolder, symbol Device:R_Small
- added U5: VXO7805-500-M, custom:VXO78x-500-M, symbol custom:VXO78x-500-M
- added U6: VXO7803-500-M, custom:VXO78x-500-M, symbol custom:VXO78x-500-M
- U2: value 4072 -> ESP32-POE Module; symbol connectors:ESP32-POE -> EnergyMonitor---ESP-PCB-rescue:ESP32-POE-connectors
Connections:
- net labels added: +5V, IRQ_10, IRQ_11, IRQ_12, IRQ_3, IRQ_4, IRQ_5, IRQ_6, IRQ_7, IRQ_8, IRQ_9, ~CS_10, ~CS_11, ~CS_12, ~CS_3, ~CS_4, ~CS_5, ~CS_6, ~CS_7, ~CS_8, ~CS_9
- wire segments 266 -> 314
- no-connect marks 3 -> 6
Other:
- note added: "Inductors: SRU8028-470Y"
- note removed: "ESP Module provides \n5V -> 3.3V conversion"
- moved on the sheet: J1, R2, U1A

Commit message: Updates! I keep adding features.
Parts:
- removed C1, C10, C11, C2, C3: 0.1 uF, Capacitor_SMD:C_0603_1608Metric_Pad1.05x0.95mm_HandSolder, symbol Device:C_Small
- removed C12, C13, C8, C9: 22 uF, Capacitor_SMD:C_1206_3216Metric_Pad1.42x1.75mm_HandSolder, symbol Device:C_Small
- removed C14, C4, C5: CP1, Capacitor_THT:CP_Radial_D12.5mm_P5.00mm, symbol Device:CP1
- removed C15, C16: CP1, Capacitor_THT:CP_Radial_D8.0mm_P3.50mm, symbol Device:CP1
- removed C6, C7: 10 uF, 35V, Capacitor_SMD:C_1206_3216Metric_Pad1.42x1.75mm_HandSolder, symbol Device:C_Small
- removed J1: Conn_02x05_Odd_Even, Connector_IDC:IDC-Header_2x05_P2.54mm_Vertical, symbol Connector_Generic:Conn_02x05_Odd_Even
- removed J2, J3, J4, J5, J6, J7: Conn_02x07_Odd_Even, Connector_IDC:IDC-Header_2x07_P2.54mm_Vertical, symbol Connector_Generic:Conn_02x07_Odd_Even
- removed L1, L2, L3: 47 uH, Inductor_SMD:L_Bourns-SRU8028_8.0x8.0mm, symbol Device:L_Small
- removed R1: 10K, Resistor_SMD:R_0603_1608Metric_Pad1.05x0.95mm_HandSolder, symbol Device:R_Small
- removed R2, R3: 330R, Resistor_SMD:R_0603_1608Metric_Pad1.05x0.95mm_HandSolder, symbol Device:R_Small
- removed U1, U3: 4072, Package_SO:SOIC-14_3.9x8.7mm_P1.27mm, symbol 4xxx:4072
- removed U2: ESP32-POE Module, Energy Monitor - ESP32 PCB:ESP32-POE, symbol EnergyMonitor---ESP-PCB-rescue:ESP32-POE-connectors
- removed U4: 4072, Package_SO:SOIC-24W_7.5x15.4mm_P1.27mm, symbol 74xx:74LS154
- removed U5: VXO7805-500-M, custom:VXO78x-500-M, symbol custom:VXO78x-500-M
- removed U6: VXO7803-500-M, custom:VXO78x-500-M, symbol custom:VXO78x-500-M
Connections:
- no-connect marks 6 -> 0
Other:
- note removed: "Each M90E36A consumes 23.5 mA\nWith LEDs, assume ~~75 mA/sensor board\nThat gives 450 mA maximum on 3.3V rail"
- note removed: "Inductors: SRU8028-470Y"
- moved on the sheet: H1, H2, H3, H4
