File: Hardware/KiCad/Energy Monitor - ESP32 PCB/ESP32 and Comms.sch (KiCad schematic (older format))
At the start: 39 parts, among them J1 Conn_02x05_Odd_Even, J2 Conn_02x07_Odd_Even, J3 Conn_02x07_Odd_Even, J4 Conn_02x07_Odd_Even, J5 Conn_02x07_Odd_Even, J6 Conn_02x07_Odd_Even, J7 Conn_02x07_Odd_Even, U1 4072, U2 ESP32-POE Module, U3 4072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

Commit message: Updates! I keep adding features.
Parts:
- removed C10, C11: 0.1 uF, Capacitor_SMD:C_0603_1608Metric_Pad1.05x0.95mm_HandSolder, symbol Device:C_Small
- removed C12, C13, C8, C9: 22 uF, Capacitor_SMD:C_1206_3216Metric_Pad1.42x1.75mm_HandSolder, symbol Device:C_Small
- removed C14, C4, C5: CP1, Capacitor_THT:CP_Radial_D12.5mm_P5.00mm, symbol Device:CP1
- removed C15, C16: CP1, Capacitor_THT:CP_Radial_D8.0mm_P3.50mm, symbol Device:CP1
- removed C6, C7: 10 uF, 35V, Capacitor_SMD:C_1206_3216Metric_Pad1.42x1.75mm_HandSolder, symbol Device:C_Small
- removed H1, H2, H3, H4: MountingHole, MountingHole:MountingHole_3.2mm_M3_Pad_Via, symbol Mechanical:MountingHole
- removed J1: Conn_02x05_Odd_Even, Connector_IDC:IDC-Header_2x05_P2.54mm_Vertical, symbol Connector_Generic:Conn_02x05_Odd_Even
- removed L1, L2, L3: 47 uH, Inductor_SMD:L_Bourns-SRU8028_8.0x8.0mm, symbol Device:L_Small
- removed U5: VXO7805-500-M, custom:VXO78x-500-M, symbol custom:VXO78x-500-M
- removed U6: VXO7803-500-M, custom:VXO78x-500-M, symbol custom:VXO78x-500-M
- added J10, J8, J9: Conn_01x04, Connector_PinHeader_2.54mm:PinHeader_1x04_P2.54mm_Vertical, symbol Connector_Generic:Conn_01x04
- added LCD?1: 0.96\"-SSD1306-DISP-I2C, custom:12864-DISP-I2C, symbol custom:0.96"-SSD1306-DISP-I2C
- added R4, R5: 2.2K, Resistor_SMD:R_0603_1608Metric_Pad1.05x0.95mm_HandSolder, symbol Device:R_Small
- added R6: 10K, Resistor_SMD:R_0603_1608Metric_Pad1.05x0.95mm_HandSolder, symbol Device:R_Small
- U2: symbol EnergyMonitor---ESP-PCB-rescue:ESP32-POE-connectors -> custom:ESP32-POE
Connections:
- net +3V3: now also J10.3 (Pin_3), J8.3 (Pin_3), J9.3 (Pin_3), R4.1, R5.1, R6.1
- net +5V: now also J10.4 (Pin_4), J8.4 (Pin_4), J9.4 (Pin_4), LCD?1.1 (VCC)
- net GND: now also J10.1 (Pin_1), J8.1 (Pin_1), J9.1 (Pin_1), LCD?1.2 (Gnd)
- net IRQ_10: now also U3.5; no longer U3.11
- net IRQ_11: now also U3.3; no longer U3.10
- net IRQ_12: now also U3.2; no longer U3.9
- net IRQ_7: now also U3.11; no longer U3.5
- net IRQ_8: now also U3.12; no longer U3.4
- net IRQ_9: now also U3.4; no longer U3.12
- net MISO: now also U2.13 (GPIO35); no longer U2.15 (GPIO33)
- net at U2.16 (GPIO32): now also U4.23 (A0); no longer U4.21 (A2)
- net at U2.20 (GPIO13/I2C-SDA): now also U4.21 (A2); no longer U4.23 (A0)
- net at U2.5 (GPIO0): now also LCD?1.3 (SCL), R4.2
- net at U2.7 (GPIO2/HS2_DATA0): now also LCD?1.4 (SDA), R5.2
- net at R3.2: now also U3.13; no longer U3.1
- new net: J10.2 (Pin_2), J8.2 (Pin_2), J9.2 (Pin_2), R6.2, U2.15 (GPIO33)
- new net: U3.1, U3.10, U3.9
- no-connect marks 6 -> 2
Other:
- note removed: "Each M90E36A consumes 23.5 mA\nWith LEDs, assume ~~75 mA/sensor board\nThat gives 450 mA maximum on 3.3V rail"
- note removed: "Inductors: SRU8028-470Y"
- moved on the sheet: U3A, U3B

Commit message: Progress!
Parts:
- added J11, J12: Conn_01x05, Connector_PinHeader_2.54mm:PinHeader_1x05_P2.54mm_Vertical, symbol Connector_Generic:Conn_01x05
Connections:
- net +3V3: now also J11.2 (Pin_2), J12.2 (Pin_2)
- net +5V: now also J11.1 (Pin_1), J12.1 (Pin_1)
- net GND: now also J11.5 (Pin_5), J12.5 (Pin_5)
- net IRQ_3: now also U1.11; no longer U1.12
- net IRQ_4: now also U1.12; no longer U1.11
- net IRQ_5: now also U1.9; no longer U1.10
- net IRQ_6: now also U1.10; no longer U1.9
- net at R4.2, U2.5 (GPIO0): now also LCD?1.4 (SDA), J11.4 (Pin_4), J12.4 (Pin_4); no longer LCD?1.3 (SCL)
- net at R5.2, U2.7 (GPIO2/HS2_DATA0): now also LCD?1.3 (SCL), J11.3 (Pin_3), J12.3 (Pin_3); no longer LCD?1.4 (SDA)
Other:
- moved on the sheet: R4, R5
Changed lines of the file:
@@
 	5450 3050 5450 3850
 Wire Wire Line
-	5150 3450 5850 3450
-Wire Wire Line
-	5850 3450 5850 3900
-Wire Wire Line
-	5850 3900 6300 3900
-Wire Wire Line
-	5750 4000 5750 3550
-Wire Wire Line
-	5750 3550 5150 3550
-Wire Wire Line
-	5750 4000 6300 4000
-Wire Wire Line
-	5350 2950 5350 3350
-Wire Wire Line
-	5350 3350 5150 3350
+	5150 3450 5750 3450
 Wire Wire Line
 	5350 2950 6300 2950
 Wire Wire Line
-	5150 3250 5250 3250
-Wire Wire Line
-	5250 3250 5250 2850
-Wire Wire Line
 	5250 2850 6300 2850
-Wire Wire Line
-	5150 1800 6300 1800
-Wire Wire Line
-	5150 1900 6300 1900
 Wire Wire Line
 	5150 2000 5250 2000
@@
 L Device:R_Small R4
 U 1 1 5F7794F8
+P 2750 2100
+F 0 "R4" H 2809 2146 50  0000 L CNN
+F 1 "2.2K" H 2809 2055 50  0000 L CNN
+F 2 "Resistor_SMD:R_0603_1608Metric_Pad1.05x0.95mm_HandSolder" H 2750 2100 50  0001 C CNN
+F 3 "~" H 2750 2100 50  0001 C CNN
+	1    2750 2100
+	1    0    0    -1
+$EndComp
+$Comp
+L Device:R_Small R5
+U 1 1 5F77A342
 P 2450 2100
-F 0 "R4" H 2509 2146 50  0000 L CNN
+F 0 "R5" H 2509 2146 50  0000 L CNN
 F 1 "2.2K" H 2509 2055 50  0000 L CNN
 F 2 "Resistor_SMD:R_0603_1608Metric_Pad1.05x0.95mm_HandSolder" H 2450 2100 50  0001 C CNN
 F 3 "~" H 2450 2100 50  0001 C CNN
 	1    2450 2100
-	1    0    0    -1
-$EndComp
-$Comp
-L Device:R_Small R5
-U 1 1 5F77A342
-P 2750 2100
-F 0 "R5" H 2809 2146 50  0000 L CNN
-F 1 "2.2K" H 2809 2055 50  0000 L CNN
-F 2 "Resistor_SMD:R_0603_1608Metric_Pad1.05x0.95mm_HandSolder" H 2750 2100 50  0001 C CNN
-F 3 "~" H 2750 2100 50  0001 C CNN
-	1    2750 2100
 	1    0    0    -1
 $EndComp
@@
 Wire Wire Line
 	2750 2400 2400 2400
-Wire Wire Line
-	2450 3650 2450 2300
 Connection ~ 2450 2300
 Connection ~ 2750 2400
-Wire Wire Line
-	2450 3650 2350 3650
-Wire Wire Line
-	2350 3850 2750 3850
-Wire Wire Line
-	2750 3850 2750 2400
 Wire Wire Line
 	8000 1700 8000 1850
@@
 Wire Wire Line
 	2350 4650 2850 4650
+Wire Wire Line
+	5150 3550 5850 3550
+Wire Wire Line
+	5850 3550 5850 3900
+Wire Wire Line
+	5850 3900 6300 3900
+Wire Wire Line
+	5750 4000 6300 4000
+Wire Wire Line
+	5750 3450 5750 4000
+Wire Wire Line
+	5350 2950 5350 3250
+Wire Wire Line
+	5150 3250 5350 3250
+Wire Wire Line
+	5250 2850 5250 3350
+Wire Wire Line
+	5250 3350 5150 3350
+Wire Wire Line
+	5150 1800 6300 1800
+Wire Wire Line
+	5150 1900 6300 1900
+Wire Wire Line
+	2450 3850 2350 3850
+Wire Wire Line
+	2450 2300 2450 2600
+Wire Wire Line
+	2350 3650 2750 3650
+Wire Wire Line
+	2750 3650 2750 2700
+$Comp
+L Connector_Generic:Conn_01x05 J11
+U 1 1 5F6CED99
+P 3600 2600
+F 0 "J11" H 3550 2950 50  0000 L CNN
+F 1 "Conn_01x05" H 3680 2551 50  0001 L CNN
+F 2 "Connector_PinHeader_2.54mm:PinHeader_1x05_P2.54mm_Vertical" H 3600 2600 50  0001 C CNN
+F 3 "~" H 3600 2600 50  0001 C CNN
+	1    3600 2600
+	1    0    0    -1
+$EndComp
+$Comp
+L Connector_Generic:Conn_01x05 J12
+U 1 1 5F7014EB
+P 3950 2600
+F 0 "J12" H 3900 2950 50  0000 L CNN
+F 1 "Conn_01x05" H 4030 2551 50  0001 L CNN
+F 2 "Connector_PinHeader_2.54mm:PinHeader_1x05_P2.54mm_Vertical" H 3950 2600 50  0001 C CNN
+F 3 "~" H 3950 2600 50  0001 C CNN
+	1    3950 2600
+	1    0    0    -1
+$EndComp
+$Comp
+L power:+3.3V #PWR0118
+U 1 1 5F7018CC
+P 3150 2150
+F 0 "#PWR0118" H 3150 2000 50  0001 C CNN
+F 1 "+3.3V" H 3165 2323 50  0000 C CNN
+F 2 "" H 3150 2150 50  0001 C CNN
+F 3 "" H 3150 2150 50  0001 C CNN
+	1    3150 2150
+	1    0    0    -1
+$EndComp
+$Comp
+L power:+5V #PWR0119
+U 1 1 5F71B36B
+P 3250 2250
+F 0 "#PWR0119" H 3250 2100 50  0001 C CNN
+F 1 "+5V" H 3265 2423 50  0000 C CNN
+F 2 "" H 3250 2250 50  0001 C CNN
+F 3 "" H 3250 2250 50  0001 C CNN
+	1    3250 2250
+	1    0    0    -1
+$EndComp
+Wire Wire Line
+	3250 2250 3250 2400
+Wire Wire Line
+	3250 2400 3400 2400
+Connection ~ 3400 2400
+Wire Wire Line
+	3400 2400 3750 2400
+Wire Wire Line
+	3150 2150 3150 2500
+Wire Wire Line
+	3150 2500 3400 2500
+Connection ~ 3400 2500
+Wire Wire Line
+	3400 2500 3750 2500
+$Comp
+L power:GND #PWR0120
+U 1 1 5F74F010
+P 3300 2900
+F 0 "#PWR0120" H 3300 2650 50  0001 C CNN
+F 1 "GND" H 3305 2727 50  0000 C CNN
+F 2 "" H 3300 2900 50  0001 C CNN
+F 3 "" H 3300 2900 50  0001 C CNN
+	1    3300 2900
+	1    0    0    -1
+$EndComp
+Wire Wire Line
+	3300 2900 3300 2800
+Wire Wire Line
+	3300 2800 3400 2800
+Connection ~ 3400 2800
+Wire Wire Line
+	3400 2800 3750 2800
+Wire Wire Line
+	3750 2700 3400 2700
+Connection ~ 2750 2700
+Wire Wire Line
+	2750 2700 2750 2400
+Connection ~ 3400 2700
+Wire Wire Line
+	3400 2700 2750 2700
+Wire Wire Line
+	3750 2600 3400 2600
+Connection ~ 2450 2600
+Wire Wire Line
+	2450 2600 2450 3850
+Connection ~ 3400 2600
+Wire Wire Line
+	3400 2600 2450 2600
 $EndSCHEMATC
