File: Hardware/KiCad/Energy Monitor - Sensor PCB - Bussed/Energy Monitor - Sensor PCB.sch (KiCad schematic (older format))
At the start: 19 parts, among them J1 Conn_02x05_Odd_Even, J2 Conn_02x17_Odd_Even, J3 Conn_02x14_Odd_Even, Q1 RUM002N05T2LCT-ND

Commit message: Common-bus variant of the power monitor.
Connections:
- net meter_1/SCLK renamed SCLK
- net meter_1/SDI renamed SDI
- net meter_1/SDO renamed SDO
Changed lines of the file:
@@
 Wire Wire Line
 	5600 1550 5600 1500
+Wire Wire Line
+	5600 1200 5600 1150
+Wire Wire Line
+	5600 850  5600 800
+Connection ~ 5600 1550
+Text Label 6150 4350 0    50   ~ 0
+SDI
+Text Label 6150 4450 0    50   ~ 0
+SDO
+Text Label 6150 4550 0    50   ~ 0
+SCLK
 Wire Bus Line
 	8300 2150 8300 2650
@@
 Wire Bus Line
 	8300 2650 8300 3450
-Wire Wire Line
-	5600 1200 5600 1150
-Wire Wire Line
-	5600 850  5600 800
-Connection ~ 5600 1550
 $EndSCHEMATC
