File: Hardware/KiCad/Energy Monitor - Transformer PCB/Energy Monitor - Transformer PCB.sch (KiCad schematic (older format))
At the start: 25 parts, among them J1 Conn_01x02, J10 Conn_02x05_Odd_Even, J2 Conn_01x02, J3 Conn_01x02, J4 Conn_02x05_Odd_Even, J5 Conn_02x05_Odd_Even, J6 Conn_02x05_Odd_Even, J7 Conn_02x05_Odd_Even, J8 Conn_02x05_Odd_Even, J9 Conn_02x05_Odd_Even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

Commit message: This seems to be getting progressively more complicated. Library cleanup, moved everything to my system library.
Parts:
- added C3: CP1, Capacitor_THT:CP_Radial_D12.5mm_P5.00mm, symbol Device:CP1
- added J11: Conn_02x05_Odd_Even, Connector_IDC:IDC-Header_2x05_P2.54mm_Vertical, symbol Connector_Generic:Conn_02x05_Odd_Even
- T1, T2, T3: symbol Transformer-Components:EI30-15.5 -> Energy-Monitor---Transformer-PCB-rescue:EI30-15.5-Transformer-Components
Connections:
- net +9V: now also C3.1, J11.1 (Pin_1), J11.3 (Pin_3), J11.5 (Pin_5), J11.7 (Pin_7)
- net GND: now also C3.2, J11.10 (Pin_10), J11.4 (Pin_4), J11.6 (Pin_6), J11.8 (Pin_8)
- no-connect marks 14 -> 16
Changed lines of the file:
@@
 	4250 5000 4250 5100
 $Comp
-L Transformer-Components:EI30-15.5 T3
+L Energy-Monitor---Transformer-PCB-rescue:EI30-15.5-Transformer-Components T3
 U 1 1 5F43DC6E
 P 3450 4800
@@
 $EndComp
 $Comp
-L Transformer-Components:EI30-15.5 T1
+L Energy-Monitor---Transformer-PCB-rescue:EI30-15.5-Transformer-Components T1
 U 1 1 5F43F017
 P 3400 2800
@@
 $EndComp
 $Comp
-L Transformer-Components:EI30-15.5 T2
+L Energy-Monitor---Transformer-PCB-rescue:EI30-15.5-Transformer-Components T2
 U 1 1 5F43F7AB
 P 3400 3400
@@
 Connection ~ 5550 4600
 Wire Wire Line
-	5550 4600 6300 4600
+	5550 4600 5700 4600
 Wire Wire Line
 	5550 5400 5550 5300
 Connection ~ 5550 5300
 Wire Wire Line
-	5550 5300 6200 5300
+	5550 5300 5700 5300
 $Comp
 L power:+9V #PWR01
@@
 Wire Wire Line
 	5050 6700 5050 6800
+$Comp
+L Connector_Generic:Conn_02x05_Odd_Even J11
+U 1 1 5F46D931
+P 7200 4900
+F 0 "J11" V 7250 5180 50  0000 L CNN
+F 1 "Conn_02x05_Odd_Even" H 7250 5226 50  0001 C CNN
+F 2 "Connector_IDC:IDC-Header_2x05_P2.54mm_Vertical" H 7200 4900 50  0001 C CNN
+F 3 "~" H 7200 4900 50  0001 C CNN
+	1    7200 4900
+	0    1    1    0
+$EndComp
+NoConn ~ 7000 4700
+NoConn ~ 7400 5200
+Wire Wire Line
+	6500 5300 7000 5300
+Wire Wire Line
+	7000 5300 7000 5200
+Connection ~ 6500 5300
+Wire Wire Line
+	7100 5200 7100 5300
+Wire Wire Line
+	7100 5300 7000 5300
+Connection ~ 7000 5300
+Wire Wire Line
+	7200 5200 7200 5300
+Wire Wire Line
+	7200 5300 7100 5300
+Connection ~ 7100 5300
+Wire Wire Line
+	7300 5200 7300 5300
+Wire Wire Line
+	7300 5300 7200 5300
+Connection ~ 7200 5300
+Wire Wire Line
+	7100 4700 7100 4600
+Wire Wire Line
+	7100 4600 6600 4600
+Connection ~ 6600 4600
+Wire Wire Line
+	7100 4600 7200 4600
+Wire Wire Line
+	7200 4600 7200 4700
+Connection ~ 7100 4600
+Wire Wire Line
+	7200 4600 7300 4600
+Wire Wire Line
+	7300 4600 7300 4700
+Connection ~ 7200 4600
+Wire Wire Line
+	7300 4600 7400 4600
+Wire Wire Line
+	7400 4600 7400 4700
+Connection ~ 7300 4600
+$Comp
+L Device:CP1 C3
+U 1 1 5F4E5B78
+P 5700 4950
+F 0 "C3" H 5815 4996 50  0000 L CNN
+F 1 "CP1" H 5815 4905 50  0000 L CNN
+F 2 "Capacitor_THT:CP_Radial_D12.5mm_P5.00mm" H 5700 4950 50  0001 C CNN
+F 3 "~" H 5700 4950 50  0001 C CNN
+	1    5700 4950
+	1    0    0    -1
+$EndComp
+Wire Wire Line
+	5700 4800 5700 4600
+Connection ~ 5700 4600
+Wire Wire Line
+	5700 4600 6300 4600
+Wire Wire Line
+	5700 5100 5700 5300
+Connection ~ 5700 5300
+Wire Wire Line
+	5700 5300 6200 5300
 $EndSCHEMATC

Commit message: MOAR.
Parts:
- removed T3: EI30-15.5, Energy Monitor - Transformer PCB:EI30-15.5-TH, symbol Energy-Monitor---Transformer-PCB-rescue:EI30-15.5-Transformer-Components
- added T3: AHI050, custom:AHI050-TH, symbol custom:AHI050
- T1, T2: footprint Energy Monitor - Transformer PCB:EI30-15.5-TH -> custom:EI30-15.5-TH; symbol Energy-Monitor---Transformer-PCB-rescue:EI30-15.5-Transformer-Components -> custom:EI30-15.5
Connections:
- wire segments 205 -> 213
Other:
- moved on the sheet: J3
Changed lines of the file:
@@
-$EndComp
-$Comp
-L Device:D D3
-U 1 1 5F44603A
-P 4500 5100
-F 0 "D3" H 4500 5317 50  0000 C CNN
-F 1 "D" H 4500 5226 50  0000 C CNN
-F 2 "Diode_THT:D_DO-41_SOD81_P12.70mm_Horizontal" H 4500 5100 50  0001 C CNN
-F 3 "~" H 4500 5100 50  0001 C CNN
-	1    4500 5100
-	1    0    0    -1
 $EndComp
 $Comp
@@
 	4350 4800 4250 4800
 Wire Wire Line
-	4250 4800 4250 5000
-Wire Wire Line
-	4250 5100 4350 5100
-Wire Wire Line
 	4350 5300 4050 5300
 Wire Wire Line
-	4050 5300 4050 4850
+	4050 5300 4050 5200
 Wire Wire Line
 	4050 4600 4350 4600
@@
 	4750 4800 4650 4800
 Wire Wire Line
-	4650 5100 4750 5100
-Wire Wire Line
-	4750 5100 4750 5300
-Wire Wire Line
 	4750 5300 4650 5300
 Wire Wire Line
-	3750 4850 4050 4850
-Connection ~ 4050 4850
-Wire Wire Line
-	4050 4850 4050 4600
-Wire Wire Line
-	4250 5000 3750 5000
-Connection ~ 4250 5000
-Wire Wire Line
-	4250 5000 4250 5100
-$Comp
-L Energy-Monitor---Transformer-PCB-rescue:EI30-15.5-Transformer-Components T3
-U 1 1 5F43DC6E
-P 3450 4800
-F 0 "T3" H 3450 4933 50  0000 C CNN
-F 1 "EI30-15.5" H 3450 4650 50  0001 C CNN
-F 2 "Energy Monitor - Transformer PCB:EI30-15.5-TH" H 3450 4800 50  0001 C CNN
-F 3 "" H 3450 4800 50  0001 C CNN
-	1    3450 4800
-	1    0    0    -1
-$EndComp
-$Comp
-L Energy-Monitor---Transformer-PCB-rescue:EI30-15.5-Transformer-Components T1
+	3750 4950 4050 4950
+Wire Wire Line
+	4250 5050 3750 5050
+$Comp
+L custom:EI30-15.5 T1
 U 1 1 5F43F017
 P 3400 2800
 F 0 "T1" H 3400 2933 50  0000 C CNN
 F 1 "EI30-15.5" H 3400 2650 50  0001 C CNN
-F 2 "Energy Monitor - Transformer PCB:EI30-15.5-TH" H 3400 2800 50  0001 C CNN
+F 2 "custom:EI30-15.5-TH" H 3400 2800 50  0001 C CNN
 F 3 "" H 3400 2800 50  0001 C CNN
 	1    3400 2800
@@
 $EndComp
 $Comp
-L Energy-Monitor---Transformer-PCB-rescue:EI30-15.5-Transformer-Components T2
+L custom:EI30-15.5 T2
 U 1 1 5F43F7AB
 P 3400 3400
 F 0 "T2" H 3400 3533 50  0000 C CNN
 F 1 "EI30-15.5" H 3400 3250 50  0001 C CNN
-F 2 "Energy Monitor - Transformer PCB:EI30-15.5-TH" H 3400 3400 50  0001 C CNN
+F 2 "custom:EI30-15.5-TH" H 3400 3400 50  0001 C CNN
 F 3 "" H 3400 3400 50  0001 C CNN
 	1    3400 3400
@@
 L Connector_Generic:Conn_01x02 J3
 U 1 1 5F458980
-P 2750 4800
-F 0 "J3" H 2668 4925 50  0000 C CNN
-F 1 "Conn_01x02" H 2668 4926 50  0001 C CNN
-F 2 "Energy Monitor - Transformer PCB:WE 691411410002 - 2 Pin Wire-To-Board Terminal Block" H 2750 4800 50  0001 C CNN
-F 3 "~" H 2750 4800 50  0001 C CNN
-	1    2750 4800
+P 2550 4700
+F 0 "J3" H 2468 4825 50  0000 C CNN
+F 1 "Conn_01x02" H 2468 4826 50  0001 C CNN
+F 2 "Energy Monitor - Transformer PCB:WE 691411410002 - 2 Pin Wire-To-Board Terminal Block" H 2550 4700 50  0001 C CNN
+F 3 "~" H 2550 4700 50  0001 C CNN
+	1    2550 4700
 	-1   0    0    -1
 $EndComp
 Wire Wire Line
-	2950 4800 3150 4800
-Wire Wire Line
 	2900 3400 3100 3400
 Wire Wire Line
@@
 	3000 3650 3100 3650
 Wire Wire Line
-	2950 4900 3050 4900
-Wire Wire Line
-	3050 4900 3050 5050
-Wire Wire Line
-	3050 5050 3150 5050
+	2750 4800 2850 4800
 NoConn ~ 9100 3250
 NoConn ~ 8600 3250
@@
 Wire Wire Line
 	5700 5300 6200 5300
+$Comp
+L custom:AHI050 T3
+U 1 1 5F4D7987
+P 3450 4700
+F 0 "T3" H 3450 4833 50  0000 C CNN
+F 1 "AHI050" H 3450 4500 50  0001 C CNN
+F 2 "custom:AHI050-TH" H 3450 4700 50  0001 C CNN
+F 3 "" H 3450 4700 50  0001 C CNN
+	1    3450 4700
+	1    0    0    -1
+$EndComp
+Wire Wire Line
+	3750 5200 4050 5200
+Connection ~ 4050 4950
+Connection ~ 4050 5200
+Connection ~ 4250 5050
+Wire Wire Line
+	4250 4800 4250 5050
+Wire Wire Line
+	4050 4600 4050 4950
+Wire Wire Line
+	4050 4950 4050 5200
+Wire Wire Line
+	3750 4800 4250 4800
+Connection ~ 4250 4800
+Wire Wire Line
+	2850 4950 3150 4950
+Wire Wire Line
+	2750 4700 3000 4700
+Wire Wire Line
+	2850 5300 3150 5300
+Wire Wire Line
+	2850 4800 2850 4950
+Connection ~ 2850 4950
+Wire Wire Line
+	2850 4950 2850 5300
+Wire Wire Line
+	3150 5050 3000 5050
+Wire Wire Line
+	3000 5050 3000 4700
+Connection ~ 3000 4700
+Wire Wire Line
+	3000 4700 3150 4700
+Wire Wire Line
+	4750 5100 4750 5300
+Wire Wire Line
+	4250 5050 4250 5100
+Wire Wire Line
+	4650 5100 4750 5100
+Wire Wire Line
+	4250 5100 4350 5100
+$Comp
+L Device:D D3
+U 1 1 5F44603A
+P 4500 5100
+F 0 "D3" H 4500 5317 50  0000 C CNN
+F 1 "D" H 4500 5226 50  0000 C CNN
+F 2 "Diode_THT:D_DO-41_SOD81_P12.70mm_Horizontal" H 4500 5100 50  0001 C CNN
+F 3 "~" H 4500 5100 50  0001 C CNN
+	1    4500 5100
+	1    0    0    -1
+$EndComp
 $EndSCHEMATC
