File: Hardware/KiCad/Energy Monitor - ESP32 PCB - Bussed/ESP32 and Comms.sch (KiCad schematic (older format))
At the start: 44 parts, among them J10 Conn_01x04, J11 Conn_01x05, J12 Conn_01x05, J2 Conn_02x17_Odd_Even, J3 Conn_02x17_Odd_Even, J8 Conn_01x04, J9 Conn_01x04, U1 74LVC1G04, U2 ESP32-POE Module, U4 74LS154

Commit message: Blerp.
Parts:
- U4: value 74LS154 -> 74HC154
Changed lines of the file:
@@
 P 4700 5850
 F 0 "U4" H 4850 6800 50  0000 C CNN
-F 1 "74LS154" H 4950 6700 50  0000 C CNN
+F 1 "74HC154" H 4950 6700 50  0000 C CNN
 F 2 "Package_SO:SOIC-24W_7.5x15.4mm_P1.27mm" H 4700 5850 50  0001 C CNN
 F 3 "" H 4700 5850 50  0001 C CNN
